Commit message: varie modifiche al codice

File: Leader-Follower_Simulation/src/move_target/description/person_standing/person_standing.urdf.xacro (robot description, xacro)
@@ -4,5 +4,5 @@
     </link>
     <joint name="base" type="fixed">
-        <origin xyz="0 0 0" rpy="0 0 0"/>
+        <origin xyz="2.3 0 0" rpy="0 0 0"/>
         <parent link="world"/>
         <child link="base_link"/>
